File: kiCad/WalkieTalkiePCB/WalkieTalkiePCB.kicad_sch (KiCad schematic)
At the start: 22 parts

Commit message: Kicad
Parts:
- removed D?: LED, symbol Device:LED
- removed R?: 470, symbol Device:R
- added U1: I2S-MIC, symbol WalkieTalkie:I2S-MIC
- R1, R2, R3, R4, R5: renamed from R?; value R -> 330
- R6: renamed from R?; value R -> 2k
- R7: renamed from R?; value R -> 2k2
- gave numbers to parts that had none: 13
Connections:
- net at R1.1, R2.1, R3.1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: now also U2.GND, U1.1 (GND)
- net at SW1.1, SW2.1, SW3.1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: now also U2.VIN, U1.2 (VCC)
- net at U2.+: now also LS1.1
- net at U2.-: now also LS1.2
