File: kiCad/WalkieTalkiePCB/WalkieTalkiePCB.kicad_sch (KiCad schematic)
At the start: 21 parts, among them SW1 SW_Push, SW2 SW_Push, SW3 SW_Push, SW4 SW_Push, SW5 SW_Push, U1 I2S-MIC, U2 3006-ADA_Adafruit_, U3 WROOM-32_DEVKITV1, U4 OLED_DISPLAY, U5 BAT-C-10TYPEC, U6 PSM-301, U7 PBS-LED-1606WH-L

Commit message: Updated PCB schematic
Parts:
- R1, R2, R3, R4, R5: value R -> 330
- R6: value R -> 2k2
- R7: value R -> 2k
- SW1: value SW_Push -> UP
- SW2: value SW_Push -> DWN
- SW3: value SW_Push -> MODE
- SW4: value SW_Push -> TLK
- SW5: value SW_Push -> XTRA
Connections:
- net GND: now also U1. (WS), U2.GAIN
- net at U4.SCL: now also U3.D22
- net at U4.SDA: now also U3.D21
- net at U1.3 (SD): now also U3.D33
- net at U2.BLCK: now also U1. (WS), U3.D32
- net at U2.DIN: now also U3.D14
- net at U2.LRC: now also U1. (WS), U3.D25
- net at R4.2, SW4.2: now also U3.D27
- net at R3.2, SW3.2: now also U3.D26
- net at R6.2, R7.1: now also U3.D34; no longer U3.D2
- net at R5.2, SW5.2: now also U3.D35
- no-connect marks 30 -> 20
Other:
- moved on the sheet: LS1, R1, R2, R3, R4, R5, SW1, SW2, SW3, SW4, SW5, U1
