File: kiCad/WalkieTalkiePCB/WalkieTalkiePCB.kicad_pcb (KiCad board)
At the start: 2 copper layers, 7 parts, among them U1 I2S-MIC, U2 3006-ADA_Adafruit_, U5 BAT-C-10TYPEC, U6 PSM-301, U7 PBS-LED-1606WH-L

Commit message: PCB
Parts:
- added R1: 330, Resistor_THT:R_Axial_DIN0207_L6.3mm_D2.5mm_P10.16mm_Horizontal, F.Cu at (217.2, 86.4)
- added R2: 330, Resistor_THT:R_Axial_DIN0207_L6.3mm_D2.5mm_P10.16mm_Horizontal, F.Cu at (217.2, 80.9)
- added R3: 330, Resistor_THT:R_Axial_DIN0207_L6.3mm_D2.5mm_P10.16mm_Horizontal, F.Cu at (205.7, 132.7)
- added R4: 330, Resistor_THT:R_Axial_DIN0207_L6.3mm_D2.5mm_P10.16mm_Horizontal, F.Cu at (217.2, 75.9)
- added R5: 330, Resistor_THT:R_Axial_DIN0207_L6.3mm_D2.5mm_P10.16mm_Horizontal, F.Cu at (217.2, 71.1)
- added R6: 2K, Resistor_THT:R_Axial_DIN0207_L6.3mm_D2.5mm_P10.16mm_Horizontal, F.Cu at (210.8, 132.7)
- added R7: 2K2, Resistor_THT:R_Axial_DIN0207_L6.3mm_D2.5mm_P10.16mm_Horizontal, F.Cu at (215.9, 132.7)
- added SW1: UP, ESP32-Walkie-Talkie-Footprints-Remaster:PUSH-BUTTON-CONTACTS, F.Cu at (168.3, 106.7)
- added SW2: DWN, ESP32-Walkie-Talkie-Footprints-Remaster:PUSH-BUTTON-CONTACTS, F.Cu at (168.3, 117.4)
- added SW3: MODE, ESP32-Walkie-Talkie-Footprints-Remaster:PUSH-BUTTON-CONTACTS, F.Cu at (217.8, 111.2)
- added SW4: TLK, ESP32-Walkie-Talkie-Footprints-Remaster:PUSH-BUTTON-CONTACTS, F.Cu at (185.5, 55.3)
- added SW5: XTRA, ESP32-Walkie-Talkie-Footprints-Remaster:PUSH-BUTTON-CONTACTS, F.Cu at (174.1, 55.3)
- added U3: PBS-LED-1606WH-L_(Toggle_Button), ESP32-Walkie-Talkie-Footprints-Remaster:PBS-LED-1606WH-L-Toggle-Switch, F.Cu at (212.7, 108.0)
- added U4: I2S-128X64-OLED-LCD_, ESP32-Walkie-Talkie-Footprints-Remaster:I2S-128x64-OLED-LCD, F.Cu at (188.9, 65.2)
- BT1: footprint ESP32 Walkie-Talkie:Battery-Contacts -> ESP32-Walkie-Talkie-Footprints-Remaster:BATTERY-CONTACTS
- LS1: footprint ESP32 Walkie-Talkie:Speaker -> ESP32-Walkie-Talkie-Footprints-Remaster:SPEAKER
- U1: value I2S-MIC -> BAT-C-10TYPEC_(BMS); footprint ESP32 Walkie-Talkie:I2S-Mic -> ESP32-Walkie-Talkie-Footprints-Remaster:BAT-C-10TYPEC-BMS
- U2: value 3006-ADA_Adafruit_ -> PSM-301-Voltage-Regulator; footprint ESP32 Walkie-Talkie:Amplifier -> ESP32-Walkie-Talkie-Footprints-Remaster:PSM-301-Voltage-Regulator
- U5: value BAT-C-10TYPEC -> I2S-INMP441_(MIC); footprint ESP32 Walkie-Talkie:USBC-BMS -> ESP32-Walkie-Talkie-Footprints-Remaster:I2SINMP441-MIC
- U6: value PSM-301 -> Amplifier; footprint ESP32 Walkie-Talkie:Voltage-Regulator -> ESP32-Walkie-Talkie-Footprints-Remaster:Amplifier; moved to B.Cu
- U7: value PBS-LED-1606WH-L -> ESP-WROOM-32; footprint ESP32 Walkie-Talkie:PBS-Button -> esp32_devkit_v1_doit:esp32_devkit_v1_doit; moved to B.Cu
- moved LS1 93.3 mm to (212.8, 62.8)
- moved U5 78.1 mm to (208.9, 142.2)
- moved U1 63.4 mm to (179.5, 123.3)
- moved U2 61.8 mm to (181.0, 94.8)
- moved U7 42.0 mm to (188.0, 104.8)
- moved U6 35.5 mm to (196.8, 71.8), turned to 180 degrees
- moved BT1 13.0 mm to (171.4, 69.1)
Other:
- board outline added: 55 x 98 mm
- board text added: "JLCJLCJLC"
- board text added: "TEJ-4M1 | Colin Jack & Filip Dumitru"

Commit message: PCB
Why do we live. Just to suffer.
Parts:
- added G***: LOGO, LOGO, B.Cu at (203.2, 60.3)
- added REF**: OSHW-Symbol_6.7x6mm_SilkScreen, Symbol:OSHW-Symbol_6.7x6mm_SilkScreen, B.Cu at (170.8, 57.1)
Connections:
- U7 pad 29: unconnected-(U7-Pad29) -> GND
- U7 pad 30: unconnected-(U7-Pad30) -> VCC
Routing:
- net VCC: track 0.00 -> 231.5 mm, vias 0 -> 3
- net GND: track 0.00 -> 228.9 mm, vias 0 -> 5
- net Net-(R4-Pad2): track 0.00 -> 100.9 mm, vias 0 -> 1
- net Net-(R5-Pad2): track 0.00 -> 98.7 mm, vias 0 -> 1
- net Net-(U5-Pad2): track 0.00 -> 86.9 mm, vias 0 -> 2
- net Net-(R2-Pad2): track 0.00 -> 68.8 mm, vias 0 -> 2
- net Net-(R1-Pad2): track 0.00 -> 53.2 mm, vias 0 -> 1
- net Net-(U2-Pad5): track 0.00 -> 33.9 mm, vias 0 -> 1
- net Net-(R3-Pad2): track 0.00 -> 18.2 mm, vias 0 -> 1
